File: Teensy_MainPCB_V1.01/TeensyPCB.kicad_pcb (KiCad board)
At the start: 2 copper layers, 141.9 x 100 mm, 68 parts, among them J1 ODO_Left, J10 Sonar_R, J11 Cutter, J12 Sonar_L, J13 P_Right, J14 Buzzer, J15 Button, J16 Power_PCB1, J17 Power_PCB2, J18 Free01_02, J19 P_Left, J2 I2C2_0, J20 Can3, J21 Ser5, J22 FreeA16_A17, J23 ESP RFID1, J24 ESP RFID2, J25 5V IN, J26 ESP32 I2C, J27 ESP32 Sens1, J28 ESP32 FREE, J29 3.3V IN, J3 I2C0_0, J30 I2C1_0, J31 Ser3, J32 ESP32 Sens2, J33 ESP32 I2C/SER, J34 Teensy On/Off, J4 I2C1_1, J5 Bumper, J6 ODO_Right, J7 Motor_Right1, J8 Motor_Left1, J9 Rain, U2 GY-521, U3 Teensy4.1, U4 ESP32-DEVKIT-V1

Commit message: Small Changes in Layout Text
Parts:
- J1 ODO_Left: renamed from J1
- J10 Sonar_R: renamed from J10
- J11 Cutter Motor: renamed from J11
- J12 Sonar_L: renamed from J12
- J13 P_Right: renamed from J13
- J14 Buzzer: renamed from J14
- J15 Button: renamed from J15
- J16 Power_PCB1: renamed from J16
- J17 Power_PCB2: renamed from J17
- J18 Free01_02: renamed from J18
- J19 P_Left: renamed from J19
- J2 I2C2_0: renamed from J2
- J20 Can3: renamed from J20
- J21 Ser5: renamed from J21
- J22 FreeA16_A17: renamed from J22
- J23 ESP RFID1: renamed from J23
- J24 ESP RFID2: renamed from J24
- J26 ESP I2C: renamed from J26
- J27 ESP Sens1: renamed from J27
- J28 ESP FREE: renamed from J28
- J3 I2C0_0: renamed from J3
- J30 I2C1_0: renamed from J30
- J31 Ser3: renamed from J31
- J32 ESP Sens2: renamed from J32
- J33 ESP I2C/SER: renamed from J33
- J34 On/Off: renamed from J34
- J4 I2C1_1: renamed from J4
- J5 Bumper: renamed from J5
- J6 ODO_Right: renamed from J6
- J7 Motor_Right1: renamed from J7
- J8 Motor_Left1: renamed from J8
- J9 Rain: renamed from J9
- JP1 Jumper_3.3V: renamed from JP1
- JP3 MotorPower: renamed from JP3
- JP5 CutterPower: renamed from JP5
- R10, R8: value 2KO -> 1.5KO
- R12, R13: value 2KO -> 1,5KO
Connections:
- J24 ESP RFID2 pad 5: unconnected-(J24-Pad5) -> (no net)
- R10 pad 1: pinPerimeterLeft -> Net-(J19-Pad3)
- R12 pad 1: GND -> Net-(J1-Pad1)
- R12 pad 2: pinOdometryRight -> GND
- R13 pad 1: GND -> Net-(J6-Pad1)
- R13 pad 2: pinOdometryLeft -> GND
- R7 pad 2: Net-(R7-Pad2) -> pinPerimeterRight
- R8 pad 1: Net-(R7-Pad2) -> Net-(J13-Pad3)
- U2 pad 5: unconnected-(U2-Pad5) -> (no net)
- U2 pad 6: unconnected-(U2-Pad6) -> (no net)
- U2 pad 7: unconnected-(U2-Pad7) -> (no net)
- U2 pad 8: unconnected-(U2-Pad8) -> (no net)
- U3 pad 1: unconnected-(U3-Pad1) -> (no net)
- U3 pad 15: unconnected-(U3-Pad15) -> (no net)
- U3 pad 34: unconnected-(U3-Pad34) -> (no net)
- U3 pad 49: unconnected-(U3-Pad49) -> (no net)
- U3 pad 51: unconnected-(U3-Pad51) -> (no net)
- U3 pad 53: unconnected-(U3-Pad53) -> (no net)
- U3 pad 55: unconnected-(U3-Pad55) -> (no net)
- U3 pad 56: unconnected-(U3-Pad56) -> (no net)
- U3 pad 57: unconnected-(U3-Pad57) -> (no net)
- U3 pad 58: unconnected-(U3-Pad58) -> (no net)
- U3 pad 59: unconnected-(U3-Pad59) -> (no net)
- U3 pad 60: unconnected-(U3-Pad60) -> (no net)
- U3 pad 61: unconnected-(U3-Pad61) -> (no net)
- U3 pad 62: unconnected-(U3-Pad62) -> (no net)
- U3 pad 63: unconnected-(U3-Pad63) -> (no net)
- U3 pad 64: unconnected-(U3-Pad64) -> (no net)
- U3 pad 65: unconnected-(U3-Pad65) -> (no net)
- U3 pad 66: unconnected-(U3-Pad66) -> (no net)
- U3 pad 67: unconnected-(U3-Pad67) -> (no net)
- U4 pad 1: unconnected-(U4-Pad1) -> (no net)
- U4 pad 10: unconnected-(U4-Pad10) -> (no net)
- U4 pad 17: unconnected-(U4-Pad17) -> (no net)
- U4 pad 19: unconnected-(U4-Pad19) -> (no net)
- U4 pad 2: unconnected-(U4-Pad2) -> (no net)
- U4 pad 23: unconnected-(U4-Pad23) -> (no net)
- U4 pad 3: unconnected-(U4-Pad3) -> (no net)
Routing:
- net pinPerimeterRight: track 0.00 -> 72.2 mm
- net Net-(R7-Pad2): track 72.2 -> 0.00 mm
Other:
- board text added: "T-MOW Teensy PCB v1.02 By B.B & S.D 11.2021"
