File: Teensy_MainPCB_V1.03/Teensy_MainPCB.sch (KiCad schematic (older format))
At the start: 68 parts, among them J1 ODO_Right, J10 Sonar_R, J11 Cutter, J12 Sonar_L, J13 P_Right, J14 Buzzer, J15 Button, J16 Power_PCB1, J17 Power_PCB2, J18 Free01_02, J19 P_Left, J2 I2C2_0, J20 Can3, J21 Ser5, J22 FreeA16_A17, J23 ESP RFID1, J24 ESP RFID2, J25 5V IN, J26 ESP32 I2C, J27 ESP32 Sens1, J28 ESP32 FREE, J29 3.3V IN, J3 I2C0_0, J30 I2C1_0, J31 Ser3, J32 ESP32 Sens2, J33 ESP32 I2C/SER, J34 Teensy On/Off, J4 I2C1_1, J5 Bumper, J6 ODO_Left, J7 Motor_Right1, J8 Motor_Left1, J9 Rain, U2 GY-521, U3 Teensy4.1, U4 ESP32-DEVKIT-V1

Commit message: Add Schematic PDF
Parts:
- D2: symbol Ardumower-rescue:LED-Zimprich -> Device:LED
- SP1: symbol Ardumower-rescue:SPEAKER-Lötpad_2,5mm -> Device:Speaker
Connections:
- wire segments 148 -> 149
Changed lines of the file:
@@
 	0    -1   -1   0
 $EndComp
-Wire Wire Line
-	2950 850  2800 850
 $Comp
 L power:GND #PWR042
@@
 $EndComp
 $Comp
-L Ardumower-rescue:LED-Zimprich D2
+L Device:LED D2
 U 1 1 608BB0E1
 P 2600 850
@@
 $EndComp
 $Comp
-L Ardumower-rescue:SPEAKER-Lötpad_2,5mm SP1
+L Device:Speaker SP1
 U 1 1 607B6900
-P 9715 5855
-F 0 "SP1" H 9993 5916 70  0000 L CNN
-F 1 "SPEAKER" H 9993 5795 70  0000 L CNN
-F 2 "Zimprich:Buzzer_12x9.5RM7.6" H 9715 5855 60  0001 C CNN
-F 3 "" H 9715 5855 60  0000 C CNN
-	1    9715 5855
-	1    0    0    -1
-$EndComp
-Text GLabel 9415 5955 0    50   Input ~ 0
+P 9765 5755
+F 0 "SP1" H 10043 5816 70  0000 L CNN
+F 1 "SPEAKER" H 10043 5695 70  0000 L CNN
+F 2 "Zimprich:Buzzer_12x9.5RM7.6" H 9765 5755 60  0001 C CNN
+F 3 "" H 9765 5755 60  0000 C CNN
+	1    9765 5755
+	1    0    0    -1
+$EndComp
+Text GLabel 9565 5855 0    50   Input ~ 0
 pinBuzzer
 $Comp
 L power:GND #PWR035
 U 1 1 60932E8B
-P 9415 5755
-F 0 "#PWR035" H 9415 5505 50  0001 C CNN
-F 1 "GND" V 9420 5627 50  0000 R CNN
-F 2 "" H 9415 5755 50  0001 C CNN
-F 3 "" H 9415 5755 50  0001 C CNN
-	1    9415 5755
+P 9565 5755
+F 0 "#PWR035" H 9565 5505 50  0001 C CNN
+F 1 "GND" V 9570 5627 50  0000 R CNN
+F 2 "" H 9565 5755 50  0001 C CNN
+F 3 "" H 9565 5755 50  0001 C CNN
+	1    9565 5755
 	0    1    1    0
 $EndComp
@@
 	1065 2595 965  2595
 Connection ~ 965  2595
+Wire Wire Line
+	2400 850  2450 850
+Wire Wire Line
+	2750 850  2950 850
 $EndSCHEMATC
