File: Teensy_MainPCB_V1.03/Teensy_MainPCB.sch (KiCad schematic (older format))
At the start: 68 parts, among them J1 ODO_Right, J10 Sonar_R, J11 Cutter, J12 Sonar_L, J13 P_Right, J14 Buzzer, J15 Button, J16 Power_PCB1, J17 Power_PCB2, J18 Free01_02, J19 P_Left, J2 I2C2_0, J20 Can3, J21 Ser5, J22 FreeA16_A17, J23 ESP RFID1, J24 ESP RFID2, J25 5V IN, J26 ESP32 I2C, J27 ESP32 Sens1, J28 ESP32 FREE, J29 3.3V IN, J3 I2C0_0, J30 I2C1_0, J31 Ser3, J32 ESP32 Sens2, J33 ESP32 I2C/SER, J34 Teensy On/Off, J4 I2C1_1, J5 Bumper, J6 ODO_Left, J7 Motor_Right1, J8 Motor_Left1, J9 Rain, U2 GY-521, U3 Teensy4.1, U4 ESP32-DEVKIT-V1

Commit message: Removed unused
Remove unused Items and sorting new
Parts:
- removed D2: LED_3V, LED_THT:LED_D3.0mm, symbol Device:LED
- removed D8: 1N5819, Diode_THT:D_DO-41_SOD81_P10.16mm_Horizontal, symbol Diode:1N5819
- removed J14: Buzzer, Connector_JST:JST_XH_B3B-XH-A_1x03_P2.50mm_Vertical, symbol Connector:Screw_Terminal_01x03
- removed J29: 3.3V IN, TerminalBlock:TerminalBlock_bornier-2_P5.08mm, symbol Connector:Screw_Terminal_01x02
- removed JP1: Jumper_3.3V, Connector_PinSocket_2.54mm:PinSocket_1x03_P2.54mm_Vertical, symbol Device:Jumper_NC_Dual
- removed R11: 100, Resistor_THT:R_Axial_DIN0207_L6.3mm_D2.5mm_P2.54mm_Vertical, symbol Device:R
- U2: symbol teensy:GY-521 -> Teensy_MainPCB-rescue:GY-521-teensy
- U3: symbol teensy:Teensy4.1 -> Teensy_MainPCB-rescue:Teensy4.1-teensy
- U4: symbol teensy:ESP32-DEVKIT-V1 -> Teensy_MainPCB-rescue:ESP32-DEVKIT-V1-teensy
Connections:
- net +3V3: now also U3.15 (3V3)
- net GND: now also U2.7 (AD0), U3.1 (GND), U3.34 (GND), U4.17 (GND)
- net pinPerimeterRight: now also R7.2, R8.1
- no-connect marks 32 -> 28
Other:
- moved on the sheet: J19, R10, R14, R9
