File: Power_PCB_v106/charge_pcb.kicad_pcb (KiCad board)
At the start: 2 copper layers, 128.1 x 64 mm, 48 parts, among them J1 Main_PCB2, J10 M Left + Mot_Left, J11 DC/DC1 DC/DC1, J12 DC/DC2 DC/DC2, J2 BAT Battery, J3 SWITCH Power Switch, J4 Mow3 + Mow3, J5 Main_PCB1, J6 Mow2 + Mow2, J7 Mow1 + Mow1, J8 Start, J9 M Right + Mot_Right, Q1 BC547C, Q2 IRF9540N, Q3 BC547C, Q4 IRF9540N, U1 CHARGE CURRENT INA226, U2 Mot Left Current INA226, U3 Mow3 Current INA226, U4 Mow2 Current INA226, U5 Mow1 Current INA226, U6 Mot Right Current INA226

Commit message: Small Changes in Labelling
Other:
- net class +24V added: clearance 0.55, trace_width 1.5, via_dia 0.8, via_drill 0.4
- net class +3V added: clearance 0.254, trace_width 0.5, via_dia 0.8, via_drill 0.4
- net class Default added: clearance 0.254, trace_width 0.254, via_dia 0.8, via_drill 0.4

Commit message: Don' know anymore
Other:
- net class +24V removed
- net class +3V removed
- net class Default removed
