File: Power_PCB_v107/charge_pcb.sch (KiCad schematic (older format))
At the start: 48 parts, among them J1 Main_PCB2, J10 Mot_Left, J11 DC/DC1, J12 DC/DC2, J2 Battery, J3 Power Switch, J4 Mow3, J5 Main_PCB1, J6 Mow2, J7 Mow1, J8 Start, J9 Mot_Right, Q1 BC547C, Q2 IRF9540N, Q3 BC547C, Q4 IRF9540N, U1 INA226, U2 INA226, U3 INA226, U4 INA226, U5 INA226, U6 INA226

Commit message: Wifi Sender Update Label
Parts:
- removed D3: NOT USE, Diode_THT:D_DO-35_SOD27_P7.62mm_Horizontal, symbol Diode:1N4148
