File: Power_PCB_v100small/charge_pcb.kicad_pcb (KiCad board)
At the start: 2 copper layers, 128.1 x 64 mm, 71 parts, among them J10 Mot_Left, J11 DC/DC1, J12 DC/DC2, J2 Main_PCB1, J4 Battery, J5 Main_PCB2, J6 Power Switch, J7 Mow1, J8 Mot_Right, J9 Start, Q1 BC547C, Q2 IRF9540N, Q3 BC547C, Q4 IRF9540N, U3 INA Charge, U4 INA226, U5 INA226, U6 INA226

Commit message: Changes
Parts:
- removed J2: Main_PCB1, Connector_JST:JST_XH_B6B-XH-A_1x06_P2.50mm_Vertical
- removed kibuzzard-630F6337: G***, kibuzzard-630F6337
- removed kibuzzard-630F6348: G***, kibuzzard-630F6348
- removed kibuzzard-630FA596: G***, kibuzzard-630FA596
- removed kibuzzard-630FA5B5: G***, kibuzzard-630FA5B5
- removed kibuzzard-630FA5E0: G***, kibuzzard-630FA5E0
- removed kibuzzard-630FA5FF: G***, kibuzzard-630FA5FF
- removed kibuzzard-6311B724: G***, kibuzzard-6311B724
- removed kibuzzard-6311B760: G***, kibuzzard-6311B760
- added J1: MainPCB, Connector_JST:JST_XH_B4B-XH-A_1x04_P2.50mm_Vertical, F.Cu at (88.6, 112.5)
- added REF**: OSHW-Logo2_7.3x6mm_SilkScreen, Symbol:OSHW-Logo2_7.3x6mm_SilkScreen, F.Cu at (104.9, 120.7)
- added REF**: ESD-Logo_6.6x6mm_SilkScreen, Symbol:ESD-Logo_6.6x6mm_SilkScreen, F.Cu at (96.3, 120.4)
- added REF**: WEEE-Logo_5.6x8mm_SilkScreen, Symbol:WEEE-Logo_5.6x8mm_SilkScreen, F.Cu at (104.6, 112.3)
- added kibuzzard-65C5049A: G***, kibuzzard-65C5049A, F.Cu at (118.6, 89.7)
- added kibuzzard-65C504B9: G***, kibuzzard-65C504B9, F.Cu at (121.2, 89.7)
- F1: value Polyfuse 5A -> 5A; footprint Fuse:Fuse_Littelfuse-LVR100 -> Zimprich:Fuseholder_Reichelt_PL112000
- F2: value Polyfuse 10A -> 10A; footprint Fuse:Fuse_Littelfuse-LVR100 -> Zimprich:Fuseholder_Reichelt_PL112000
- moved D4 39.5 mm to (194.9, 93.2)
- moved kibuzzard-630F6257 32.4 mm to (123.1, 123.5)
- moved J7 32.4 mm to (125.6, 117.9)
- moved U4 32.4 mm to (122.4, 101.9)
- moved D8 32.4 mm to (115.1, 120.9)
- moved kibuzzard-630FA55C 31.5 mm to (145.0, 89.7)
- moved U5 29.0 mm to (148.8, 101.9)
- moved kibuzzard-62B75EB1 29.0 mm to (149.6, 123.2)
- moved D9 29.0 mm to (141.6, 120.9)
- moved J8 29.0 mm to (152.1, 117.6)
- moved kibuzzard-630FA573 26.4 mm to (147.6, 89.7)
- moved kibuzzard-630FA52F 25.9 mm to (173.7, 89.9)
- moved R5 24.6 mm to (191.3, 110.7)
- moved R6 24.6 mm to (191.3, 107.2)
- moved R7 24.6 mm to (191.3, 103.6)
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Connections:
- F1 pad 1: V_CHARGE -> Net-(BT1-Pad1)
- F1 pad 2: Net-(BT1-Pad1) -> V_CHARGE
- F2 pad 1: Net-(D4-Pad1) -> Net-(J6-Pad2)
- F2 pad 2: Net-(F2-Pad2) -> Net-(D4-Pad1)
- J6 pad 2: Net-(F2-Pad2) -> Net-(J6-Pad2)
- U3 pad 5: SCL0 -> SDA0
- U3 pad 6: SDA0 -> SCL0
- U4 pad 5: SCL1 -> SDA0
- U4 pad 6: SDA1 -> SCL0
- U5 pad 5: SCL0 -> SDA0
- U5 pad 6: SDA0 -> SCL0
- U6 pad 5: SCL0 -> SDA0
- U6 pad 6: SDA0 -> SCL0
Routing:
- net V_Bat: track 0.00 -> 177.5 mm
- net +3V3: track 0.00 -> 126.1 mm
- net SCL0: track 0.00 -> 116.3 mm
- net pinBatterySwitch: track 0.00 -> 110.3 mm
- net SDA0: track 0.00 -> 110.2 mm
- net V_CHARGE: track 0.00 -> 49.4 mm
- net Net-(D5-Pad1): track 0.00 -> 47.6 mm
- net Net-(JP1-Pad2): track 0.00 -> 44.3 mm
- net Net-(D4-Pad1): track 0.00 -> 43.5 mm
- net Net-(J9-Pad1): track 0.00 -> 43.2 mm
- net Net-(Q1-Pad1): track 0.00 -> 40.3 mm
- net Net-(D3-Pad1): track 0.00 -> 39.2 mm
- net Net-(Q3-Pad2): track 0.00 -> 36.4 mm
- net Net-(J4-Pad1): track 0.00 -> 30.9 mm
- net Net-(J6-Pad2): track 0.00 -> 24.9 mm
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- added copper zone on B.Cu, net GND
