File: Power_PCB_v100small/charge_pcb.kicad_sch (KiCad schematic)
At the start: 42 parts, among them J10 Mot_Left, J11 DC/DC1, J12 DC/DC2, J2 Main_PCB1, J4 Battery, J5 Main_PCB2, J6 Power Switch, J7 Mow1, J8 Mot_Right, J9 Start, Q1 BC547C, Q2 IRF9540N, Q3 BC547C, Q4 IRF9540N, U3 INA Charge, U4 INA226, U5 INA226, U6 INA226

Commit message: Changes
Parts:
- removed F1: Polyfuse 5A, Fuse:Fuse_Littelfuse-LVR100, symbol Device:Polyfuse
- removed F2: Polyfuse 10A, Fuse:Fuse_Littelfuse-LVR100, symbol Device:Polyfuse
- removed J2: Main_PCB1, Connector_JST:JST_XH_B6B-XH-A_1x06_P2.50mm_Vertical, symbol Connector:Screw_Terminal_01x06
- added F1: 5A, Zimprich:Fuseholder_Reichelt_PL112000, symbol Zimprich:FUSE
- added F2: 10A, Zimprich:Fuseholder_Reichelt_PL112000, symbol Zimprich:FUSE
- added J1: MainPCB, Connector_JST:JST_XH_B4B-XH-A_1x04_P2.50mm_Vertical, symbol Connector:Screw_Terminal_01x04
Connections:
- net SCL1 is gone; now on net SDA0: U4.5 (SDA)
- net SDA1 is gone; now on net SCL0: U4.6 (SCL)
- net +3V3: now also J1.4 (Pin_4)
- net GND: now also J1.3 (Pin_3)
- net SCL0: now also U3.6 (SCL), U5.6 (SCL), U6.6 (SCL), J1.1 (Pin_1); no longer U3.5 (SCL), U5.5 (SCL), U6.5 (SCL)
- net SDA0: now also U3.5 (SDA), U5.5 (SDA), U6.5 (SDA), J1.2 (Pin_2); no longer U3.6 (SDA), U5.6 (SDA), U6.6 (SDA)
- net V_CHARGE: now also F1.2
- net at BT1.1 (+): now also F1.1
- net at J6.2: now also F2.1
- net at D4.1 (K), D5.2 (A): now also F2.2
